File: hardware/tdlf_server/tdlf_server_top_modulaire.brd (EAGLE design)
At the start: 30 x 128.5 mm, 7 parts

Commit message: Version 0.5 ready for CV outputs
Other:
- board text added: "v 0.5"
- board text removed: "v 0.4"
Changed lines of the file:
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@@
 </layers>
 <board>
-<fusionsync huburn="a.cGVyc29uYWw6dWUyYTYyMmQz" projecturn="a.cGVyc29uYWw6dWUyYTYyMmQzIzIwMjAwMTA4MjUzMTkwODgx" f3durn="urn:adsk.wipprod:dm.lineage:EJ7CIL_8QPSL4HfMM387xA" pcbguid="" lastpulledtime="" lastsyncedchangeguid="" latestrevisionid="1e268f09-bdda-4e8c-a022-348851f8809f" lastsyncedrevisionid="1e268f09-bdda-4e8c-a022-348851f8809f" lastboardhashguid="10110adf-730a-8ede-3051-079abd0e3524" lastpushedtime="2021-04-02T02:38:33Z" linktopcb3d="false"/>
+<fusionsync huburn="a.cGVyc29uYWw6dWUyYTYyMmQz" projecturn="a.cGVyc29uYWw6dWUyYTYyMmQzIzIwMjAwMTA4MjUzMTkwODgx" f3durn="urn:adsk.wipprod:dm.lineage:EJ7CIL_8QPSL4HfMM387xA" pcbguid="" lastpulledtime="" lastsyncedchangeguid="" latestrevisionid="1e268f09-bdda-4e8c-a022-348851f8809f" lastsyncedrevisionid="1e268f09-bdda-4e8c-a022-348851f8809f" lastboardhashguid="10110adf-730a-8ede-3051-079abd0e3524" lastpushedtime="2021-04-02T02:38:33Z" linktopcb3d="true"/>
 <plain>
 <wire x1="0" y1="-14.25" x2="0" y2="114.25" width="0.1524" layer="20"/>
@@
 <text x="6.8" y="102.2" size="1.9304" layer="29" font="vector">Technologies
 de la fête</text>
-<text x="18.6" y="102.2" size="1.016" layer="29" font="vector"> v 0.4</text>
+<text x="18.6" y="102.2" size="1.016" layer="29" font="vector"> v 0.5</text>
 <circle x="7.5" y="7.8" radius="3.25" width="0.254" layer="20"/>
 <circle x="22.8" y="7.8" radius="3.25" width="0.254" layer="20"/>
