File: hardware/tdlf_sensor/CajitaAbierta/CajitaAbierta.brd (EAGLE design)
At the start: 32.1 x 61.8 mm, 30 parts

Commit message: Testing CV Pitch out
Parts:
- moved 5V_IN 0.40 mm to (23.0, 29.0)
- moved BAT- 0.30 mm to (9.15, 28.9)
- moved GND 0.30 mm to (9.15, 47.3)
- moved BATT+ 0.30 mm to (23.0, 47.2)
Routing:
- net MOSI: track 46.4 -> 47.8 mm
